File: PinebookPro-M2-A+E-adapter.kicad_pcb (KiCad board)
At the start: 2 copper layers, 70.5 x 32 mm, 34 parts, among them J1 Conn_01x35_MountingPin, J2 M.2-NGFF-A+E-Key, U1 TPS63001

Commit message: Add bom
Parts:
- C1, C5: value C -> DNP
- R3, R4: value R -> 330 R
Changed lines of the file:
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@@
       (rotate (xyz 0 0 0))
     )
-    (model ${KIPRJMOD}/lib/DRC0010J.stp
+    (model ${KIPRJMOD}/lib/3rdparty/DRC0010J.stp
       (at (xyz 0 0 0))
       (scale (xyz 1 1 1))
@@
     (pad 1 smd rect (at -5.1 1.4 90) (size 0.3 0.8) (layers F.Cu F.Paste F.Mask)
       (net 1 GND))
-    (model ${KIPRJMOD}/lib/ffc-closed.step
+    (model ${KIPRJMOD}/lib/3rdparty/ffc-closed.step
       (at (xyz 0 0 0))
       (scale (xyz 1 1 1))
@@
       (effects (font (size 1 1) (thickness 0.15)))
     )
-    (fp_text value R (at 0 1.65 90) (layer F.Fab)
+    (fp_text value "330 R" (at 0 1.65 90) (layer F.Fab)
       (effects (font (size 1 1) (thickness 0.15)))
     )
@@
       (effects (font (size 1 1) (thickness 0.15)))
     )
-    (fp_text value R (at 0 1.65 90) (layer F.Fab)
+    (fp_text value "330 R" (at 0 1.65 90) (layer F.Fab)
       (effects (font (size 1 1) (thickness 0.15)))
     )
@@
       (rotate (xyz 0 0 0))
     )
-    (model ${KIPRJMOD}/lib/Coilcraft-XAL4020.step
+    (model ${KIPRJMOD}/lib/3rdparty/Coilcraft-XAL4020.step
       (at (xyz 0 0 0))
       (scale (xyz 1 1 1))
@@
     (pad "" np_thru_hole circle (at -10 0 270) (size 1.1 1.1) (drill 1.1) (layers *.Cu *.Mask))
     (pad "" np_thru_hole circle (at 10 0 270) (size 1.6 1.6) (drill 1.6) (layers *.Cu *.Mask))
-    (model ${KIPRJMOD}/lib/m.2-connector.stp
+    (model ${KIPRJMOD}/lib/3rdparty/m.2-connector.stp
       (offset (xyz 0 -2.5 2))
       (scale (xyz 1 1 1))
@@
       (effects (font (size 1 1) (thickness 0.15)))
     )
-    (fp_text value C (at 0 1.82 90) (layer F.Fab)
+    (fp_text value DNP (at 0 1.82 90) (layer F.Fab)
       (effects (font (size 1 1) (thickness 0.15)))
     )
@@
       (effects (font (size 1 1) (thickness 0.15)))
     )
-    (fp_text value C (at 0 1.82 90) (layer F.Fab)
-      (effects (font (size 1 1) (thickness 0.15)))
-    )
+    (fp_text value DNP (at 0 1.82 90) (layer F.Fab)
+      (effects (font (size 1 1) (thickness 0.15)))
+    )
